File: QL_GST_Rom_board.kicad_sch (KiCad schematic)
At the start: 18 parts, among them J1 QL_SLOT_DIN41612, Q1 PN2222A, SW1 SW_DP3T, U1 27128, U2 27128, U3 27128, U4 27128, U5 74LS139, U6 74LS12, U7 74LS27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

Commit message: probably good schematic
Parts:
- U1, U2, U3, U4: footprint Package_DIP:DIP-28_W15.24mm -> Package_DIP:DIP-28_W15.24mm_Socket_LongPads
Connections:
- net A14: no longer U8.3 (C)
- net A16: no longer U7.2
- net A18: now also U7.2; no longer U6.11
- net CLKCPU: now also U8.11 (C)
- net RESET: now also U8.3 (C); no longer U8.11 (C)
- net RW: now also U6.11; no longer U7.4
- net VCC: now also U5.2 (A0), U5.3 (A1), U6.2, U6.3, U6.4; no longer U8.13 (~{R})
- net at U8.9 (Q): now also U6.13; no longer SW1.2
- net SW1_C: now reaches SW1.3, U8.2 (D)
- net SW1_C: now also SW1.7
- net at U7.5, U8.5 (Q): now also U7.4
- net at Q1.2 (B), U6.5, U7.6: now also U8.12 (D), U8.13 (~{R}); no longer U6.3, U6.4
- net SW1_6: now reaches SW1.6
- net SW1_6: now also SW1.2
- net at U8.8 (~{Q}): no longer U8.12 (D)
Other:
- moved on the sheet: R1, SW1B, U6A, U6B, U8B

Commit message: small fix
Parts:
- C1, C3, C4: value C -> 100n
- C2: value C_Polarized -> 22uF/16V
- R1: value 10k -> 2K2; footprint Resistor_THT:R_Axial_DIN0207_L6.3mm_D2.5mm_P7.62mm_Horizontal -> Resistor_THT:R_Axial_DIN0207_L6.3mm_D2.5mm_P15.24mm_Horizontal
- R2: value 10k -> 2K2; footprint Resistor_THT:R_Axial_DIN0207_L6.3mm_D2.5mm_P7.62mm_Horizontal -> Resistor_THT:R_Axial_DIN0207_L6.3mm_D2.5mm_P10.16mm_Horizontal
Other:
- title: Sinclair QL Interface Template -> Sinclair QL ROM Board
Changed lines of the file:
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@@
 	(paper "A3")
 	(title_block
-		(title "Sinclair QL Interface Template")
-		(date "2022-01-16")
+		(title "Sinclair QL ROM Board")
+		(date "2025-08-01")
 		(rev "0.0")
 		(company "Alvaro Alea Fernandez")
-		(comment 1 "Use this schematic as a template for ")
-		(comment 2 "projects of interface for sinclair QL")
-		(comment 3 "Basic Circuits and PCB Dimensions")
 	)
 	(text "LINEAR POWER SUPPLY"
@@
 			)
 		)
-		(property "Value" "C_Polarized"
+		(property "Value" "22uF/16V"
 			(at 34.29 260.3499 0)
 			(effects
@@
 			)
 		)
-		(property "Value" "C"
+		(property "Value" "100n"
 			(at 96.52 260.3499 0)
 			(effects
@@
 			)
 		)
-		(property "Value" "C"
+		(property "Value" "100n"
 			(at 62.23 260.3499 0)
 			(effects
@@
 			)
 		)
-		(property "Value" "C"
+		(property "Value" "100n"
 			(at 85.09 260.3499 0)
 			(effects
@@
 			)
 		)
-		(property "Value" "10k"
+		(property "Value" "2K2"
 			(at 156.21 152.3999 0)
 			(effects
@@
 			)
 		)
-		(property "Footprint" "Resistor_THT:R_Axial_DIN0207_L6.3mm_D2.5mm_P7.62mm_Horizontal"
+		(property "Footprint" "Resistor_THT:R_Axial_DIN0207_L6.3mm_D2.5mm_P10.16mm_Horizontal"
 			(at 151.892 151.13 90)
 			(effects
@@
 			)
 		)
-		(property "Value" "10k"
+		(property "Value" "2K2"
 			(at 203.2 156.2099 0)
 			(effects
@@
 			)
 		)
-		(property "Footprint" "Resistor_THT:R_Axial_DIN0207_L6.3mm_D2.5mm_P7.62mm_Horizontal"
+		(property "Footprint" "Resistor_THT:R_Axial_DIN0207_L6.3mm_D2.5mm_P15.24mm_Horizontal"
 			(at 198.882 154.94 90)
 			(effects

Commit message: updated and 3d model
Parts:
- Q1: footprint Package_TO_SOT_THT:TO-92_Inline -> Package_TO_SOT_THT:TO-92L_Inline_Wide
- SW1: value SW_DP3T -> SK23D05 Type 6+2
Changed lines of the file:
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@@
 			)
 		)
-		(property "Value" "SW_DP3T"
+		(property "Value" "SK23D05 Type 6+2"
 			(at 110.49 181.61 0)
 			(effects
@@
 			)
 		)
-		(property "Footprint" "Package_TO_SOT_THT:TO-92_Inline"
+		(property "Footprint" "Package_TO_SOT_THT:TO-92L_Inline_Wide"
 			(at 191.77 192.405 0)
 			(effects
@@
 			)
 		)
-		(property "Value" "SW_DP3T"
+		(property "Value" "SK23D05 Type 6+2"
 			(at 109.22 213.36 0)
 			(effects

Commit message: remove unused pins in schematic
Connections:
- net GND: now also SW1.0 (CASE)
- net O_SP0: no longer names the net of J1.a29 (SP0)
- net O_SP1: no longer names the net of J1.a28 (SP1)
- net O_SP2: no longer names the net of J1.a26 (SP2)
- net O_SP3: no longer names the net of J1.b26 (SP3)
- no-connect marks 18 -> 22
Changed lines of the file:
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@@
 	(title_block
 		(title "Sinclair QL ROM Board")
-		(date "2025-08-01")
+		(date "2025-08-23")
 		(rev "0.0")
 		(company "Alvaro Alea Fernandez")
@@
 	)
 	(junction
+		(at 102.87 196.85)
+		(diameter 0)
+		(color 0 0 0 0)
+	)
+	(junction
 		(at 152.4 245.11)
 		(diameter 0)
@@
 	)
 	(no_connect
+		(at 36.83 99.06)
+	)
+	(no_connect
+		(at 36.83 106.68)
+	)
+	(no_connect
+		(at 62.23 99.06)
+	)
+	(no_connect
 		(at 62.23 104.14)
 	)
@@
 	)
 	(no_connect
+		(at 36.83 104.14)
+	)
+	(no_connect
 		(at 36.83 109.22)
 	)
@@
 	(wire
 		(pts
-			(xy 62.23 99.06) (xy 71.12 99.06)
-		)
-		(stroke
-			(width 0)
-			(type default)
-		)
-	)
-	(wire
-		(pts
 			(xy 21.59 53.34) (xy 36.83 53.34)
 		)
@@
 	(wire
 		(pts
+			(xy 102.87 198.12) (xy 102.87 196.85)
+		)
+		(stroke
+			(width 0)
+			(type default)
+		)
+	)
+	(wire
+		(pts
 			(xy 62.23 53.34) (xy 71.12 53.34)
 		)
@@
 	(wire
 		(pts
+			(xy 102.87 190.5) (xy 105.41 190.5)
+		)
+		(stroke
+			(width 0)
+			(type default)
+		)
+	)
+	(wire
+		(pts
 			(xy 152.4 245.11) (xy 152.4 246.38)
 		)
@@
 		)
 	)
-	(wire
-		(pts
-			(xy 27.94 106.68) (xy 36.83 106.68)
-		)
-		(stroke
-			(width 0)
-			(type default)
-		)
-	)
 	(bus
 		(pts
@@
 		)
 	)
-	(wire
-		(pts
-			(xy 27.94 104.14) (xy 36.83 104.14)
-		)
-		(stroke
-			(width 0)
-			(type default)
-		)
-	)
 	(bus
 		(pts
@@
 	(wire
 		(pts
-			(xy 27.94 99.06) (xy 36.83 99.06)
-		)
-		(stroke
-			(width 0)
-			(type default)
-		)
-	)
-	(wire
-		(pts
 			(xy 265.43 73.66) (xy 275.59 73.66)
 		)
@@
 	(wire
 		(pts
+			(xy 102.87 196.85) (xy 110.49 196.85)
+		)
+		(stroke
+			(width 0)
+			(type default)
+		)
+	)
+	(wire
+		(pts
 			(xy 220.98 81.28) (xy 218.44 81.28)
 		)
@@
 	(wire
 		(pts
+			(xy 102.87 196.85) (xy 102.87 190.5)
+		)
+		(stroke
+			(width 0)
+			(type default)
+		)
+	)
+	(wire
+		(pts
 			(xy 273.05 78.74) (xy 273.05 81.28)
 		)
@@
 		)
 	)
-	(wire
-		(pts
-			(xy 101.6 190.5) (xy 105.41 190.5)
-		)
-		(stroke
-			(width 0)
-			(type default)
-		)
-	)
 	(bus
 		(pts
@@
 		)
 	)
-	(label "O_SP2"
-		(at 29.21 99.06 0)
-		(effects
-			(font
-				(size 1.27 1.27)
-			)
-			(justify left bottom)
-		)
-	)
 	(label "SW1_C"
 		(at 115.57 187.96 0)
@@
 		)
 	)
-	(label "O_SP1"
-		(at 29.21 104.14 0)
-		(effects
-			(font
-				(size 1.27 1.27)
-			)
-			(justify left bottom)
-		)
-	)
 	(label "D0"
 		(at 132.08 40.64 0)
@@
 		)
 	)
-	(label "O_SP0"
-		(at 29.21 106.68 0)
-		(effects
-			(font
-				(size 1.27 1.27)
-			)
-			(justify left bottom)
-		)
-	)
 	(label "D5"
 		(at 295.91 53.34 0)
@@
 		)
 	)
-	(label "O_SP3"
-		(at 66.04 99.06 0)
-		(effects
-			(font
-				(size 1.27 1.27)
-			)
-			(justify left bottom)
-		)
-	)
 	(label "A3"
 		(at 105.41 48.26 0)
@@
 		(pin "2"
 		)
+		(pin "0"
+		)
 		(instances
 			(project ""
@@
 	)
 	(symbol
+		(lib_name "SW_DP3T_1")
 		(lib_id "Switch:SW_DP3T")
 		(at 109.22 219.71 0)
@@
 		(pin "2"
 		)
+		(pin "0"
+		)
 		(instances
 			(project ""
@@
 	(symbol
 		(lib_id "power:GND")
-		(at 101.6 190.5 0)
+		(at 102.87 198.12 0)
 		(unit 1)
 		(exclude_from_sim no)
@@
 		(fields_autoplaced yes)
 		(property "Reference" "#PWR03"
-			(at 101.6 196.85 0)
+			(at 102.87 204.47 0)
 			(effects
 				(font
@@
 		)
 		(property "Value" "GND"
-			(at 101.6 195.58 0)
+			(at 102.87 203.2 0)
 			(effects
 				(font
@@
 		)
 		(property "Footprint" ""
-			(at 101.6 190.5 0)
+			(at 102.87 198.12 0)
 			(effects
 				(font
@@
 		)
 		(property "Datasheet" ""
-			(at 101.6 190.5 0)
+			(at 102.87 198.12 0)
 			(effects
 				(font
@@
 		)
 		(property "Description" ""
-			(at 101.6 190.5 0)
+			(at 102.87 198.12 0)
 			(effects
 				(font
